File: NeoJointsV2/NeoJointV2A-090.brd (EAGLE design)
At the start: 16.7 x 16.5 mm, 5 parts

Commit message: update neojointv2a
Parts:
- added JP4: (no value), SparkFun-Connectors:1X01
- moved JP2 2.00 mm to (8.46, 10.7)
Connections:
- net B: now also JP4.1
Routing:
- net B: track 17.7 -> 14.9 mm
Changed lines of the file:
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@@
 <attribute name="VALUE" x="7.706" y="4.305" size="1.27" layer="27"/>
 </element>
-<element name="JP2" library="SparkFun-Connectors" package="1X01" value="" x="6.857" y="9.536" smashed="yes">
-<attribute name="VALUE" x="5.587" y="6.361" size="1.27" layer="27"/>
+<element name="JP2" library="SparkFun-Connectors" package="1X01" value="" x="8.457" y="10.736" smashed="yes">
+<attribute name="VALUE" x="7.187" y="7.561" size="1.27" layer="27"/>
 </element>
 <element name="JP3" library="SparkFun-Connectors" package="1X01" value="" x="4.746" y="11.608" smashed="yes">
@@
 <element name="U$1" library="todstuff" package="LEDSTRIP-3P" value="LED_STRIP_3P" x="5.5" y="2.7" rot="R90"/>
 <element name="U$2" library="todstuff" package="LEDSTRIP-3P" value="LED_STRIP_3P" x="14" y="11"/>
+<element name="JP4" library="SparkFun-Connectors" package="1X01" value="" x="5.8" y="8.2" smashed="yes">
+<attribute name="VALUE" x="4.53" y="5.025" size="1.27" layer="27"/>
+</element>
 </elements>
 <signals>
@@
 <wire x1="8.976" y1="7.48" x2="11" y2="8.4" width="0.4064" layer="1"/>
 </signal>
-<signal name="B">
-<contactref element="JP2" pad="1"/>
-<contactref element="U$1" pad="B"/>
-<contactref element="U$2" pad="B"/>
-<wire x1="14" y1="11" x2="10.5" y2="11" width="1.4224" layer="1"/>
-<wire x1="5.5" y1="2.7" x2="5.5" y2="5.9" width="1.4224" layer="1"/>
-<wire x1="10.5" y1="11" x2="5.5" y2="5.9" width="1.4224" layer="1" curve="91.134523"/>
-<wire x1="5.5" y1="5.9" x2="6.857" y2="9.536" width="0.4064" layer="1"/>
-</signal>
 <signal name="C">
 <contactref element="JP3" pad="1"/>
@@
 <wire x1="2.8" y1="5.9" x2="4.746" y2="11.608" width="0.4064" layer="1"/>
 </signal>
+<signal name="B">
+<contactref element="U$2" pad="B"/>
+<contactref element="U$1" pad="B"/>
+<contactref element="JP2" pad="1"/>
+<contactref element="JP4" pad="1"/>
+<wire x1="8.457" y1="10.736" x2="5.8" y2="8.2" width="0.8128" layer="1" curve="-0.394947"/>
+<wire x1="5.5" y1="2.7" x2="5.5" y2="7.9" width="1.27" layer="1"/>
+<wire x1="5.5" y1="7.9" x2="5.8" y2="8.2" width="1.27" layer="1" curve="-90"/>
+<wire x1="14" y1="11" x2="8.721" y2="11" width="1.27" layer="1"/>
+<wire x1="8.721" y1="11" x2="8.457" y2="10.736" width="1.27" layer="1" curve="90"/>
+</signal>
 </signals>
